File: main.sch (EAGLE design)
At the start: 113 parts, among them IC2 X9C102S, J3 SJ-43617-SMT, J5 CAMERA-HIMAXBOTTOM-CONTACT, M1 MOTOR10MM, Q1 600mA/40V, Q3 TRANSISTOR-NPN_MUN2211, Q4 600mA/40V, U1 MCP73831, U10 V_REG_317SMD, U11 MAX17048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

Commit message: Organized schematic
Other:
- note added: "Audio Processor"
- note added: "Battery Charging and Regulation Power Managment USB-C Interface"
- note added: "Display Interface"
- note added: "Main Peripherals"
- note added: "RP2040 Processor and 8MB QSPI NOR FLASH"
- note added: "SIM808 Interface"
- moved on the sheet: B1, C1, C10, C11, C12, C13, C14, C15, C16, C17, C18, C19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
